File: Coco_Seal_hardware.kicad_sch (KiCad schematic)
At the start: 38 parts, among them J1 USB_C_Receptacle_USB2.0_14P, Q1 FS8205A, Q2 Q_NMOS, SW4 SW_Push, SW5 SW_Push, SW6 SW_Push, U1 ESP32-C3-WROOM-02-N4, U2 E220-900T22S（JP）-EV2, U3 DW01A, U5 AP2112K-3.3, U6 TP4056-42-ESOP8, U7 TPD2EUSB30A, U8 SSD1306_OLED

Commit message: フットプリント調整、基板設計開始、途中かけ
Parts:
- removed J1: USB_C_Receptacle_USB2.0_14P, symbol Connector:USB_C_Receptacle_USB2.0_14P
- removed Q2: Q_NMOS, Package_TO_SOT_SMD:SOT-23, symbol Device:Q_NMOS
- removed U1: ESP32-C3-WROOM-02-N4, ESP32-C3-WROOM-02-N4:MODULE_ESP32-C3-WROOM-02-H4, symbol ESP32-C3-WROOM-02-N4:ESP32-C3-WROOM-02-N4
- removed U2: E220-900T22S（JP）-EV2, symbol my_simbles:E220-900T22S(JP)-EV2
- added C10, C3: 470μF, easyeda2kicad:CAP-SMD_BD8.0-L8.3-W8.3-FD, symbol Device:C
- added D2: LED_Dual_KAK, LED_THT:LED_D5.0mm-3, symbol Device:LED_Dual_KAK
- added J1: E220-900T22S(JP), Connector_PinSocket_2.54mm:PinSocket_1x07_P2.54mm_Vertical, symbol Connector:Conn_01x07_Socket
- added Q3: Q_NMOS_GSD, Package_TO_SOT_SMD:SOT-23-3, symbol Transistor_FET:Q_NMOS_GSD
- added R8, R9: 1k, easyeda2kicad:R0603, symbol Device:R
- added U2: ESP32-C3-WROOM-02, RF_Module:ESP32-C3-WROOM-02, symbol RF_Module:ESP32-C3-WROOM-02
- added USB1: TYPE-C 16PIN 2MD, easyeda2kicad:USB-C-SMD_TYPE-C-16PIN-2MD-073, symbol easyeda2kicad:TYPE-C16PIN2MD
- BT1: footprint (none) -> Connector_JST:JST_PH_S2B-PH-K_1x02_P2.00mm_Horizontal
- BZ1: footprint (none) -> easyeda2kicad:BUZ-TH_BD24.3-P15.00_PKB24SPCH3601-B0
- C1: renamed from C5; footprint (none) -> easyeda2kicad:C0603
- C2: renamed from C3; footprint (none) -> easyeda2kicad:C1206
- C4: renamed from C8; footprint (none) -> easyeda2kicad:C1206
- C5: renamed from C6; footprint (none) -> easyeda2kicad:C0603
- C6: renamed from C2; footprint (none) -> easyeda2kicad:C1206
- C7: footprint (none) -> easyeda2kicad:C0603
- C8: renamed from C4; footprint (none) -> easyeda2kicad:C1206
- C9: renamed from C1; footprint (none) -> easyeda2kicad:C0603
- D1: footprint (none) -> LED_THT:LED_D5.0mm-3
- R1: renamed from R9; footprint (none) -> easyeda2kicad:R0603
- R10: renamed from R5; footprint (none) -> easyeda2kicad:R0603
- R11: renamed from R7; footprint (none) -> easyeda2kicad:R0603
- R12: renamed from R8; footprint (none) -> easyeda2kicad:R0603
- R13: renamed from R4; footprint (none) -> easyeda2kicad:R0603
- R14: renamed from R3; footprint (none) -> easyeda2kicad:R0603
- R15: renamed from R13; footprint (none) -> easyeda2kicad:R0603
- R16: renamed from R14; footprint (none) -> easyeda2kicad:R0603
- R2: renamed from R10; footprint (none) -> easyeda2kicad:R0603
- R3: renamed from R11; footprint (none) -> easyeda2kicad:R0603
- R4: renamed from R12; footprint (none) -> easyeda2kicad:R0603
- R5: renamed from R1; footprint (none) -> easyeda2kicad:R0603
- R6: renamed from R2; footprint (none) -> easyeda2kicad:R0603
- R7: renamed from R6; footprint (none) -> easyeda2kicad:R0603
- U7: renamed from U8; footprint (none) -> Connector_PinSocket_2.54mm:PinSocket_1x04_P2.54mm_Vertical
- renumbered SW4 to SW1, SW5 to SW2, SW6 to SW3, U7 to U1, U6 to U3, U3 to U6
Connections:
- net 3.3V: now also C10.1, C3.1, J1.6 (Pin_6), U2.1 (3V3)
- net 5V: now also C2.1, D2.2 (A), USB1.A4B9 (VBUS), USB1.B4A9 (VBUS); no longer C2.2
- net BATT+: now also Q3.3 (D)
- net GND: now also C1.2, C2.2, C7.2, C10.2, C3.2, J1.7 (Pin_7), U2.19 (GND), U2.9 (GND), USB1.13 (EH), USB1.14 (EH), USB1.A1B12 (GND), USB1.B1A12 (GND); no longer C1.1, C2.1, C7.1, U3.6 (~{STDBY}), U3.7 (~{CHRG})
- net GPIO0: now also C7.1, U2.18 (IO0); no longer C7.2
- net GPIO1: now also U2.17 (IO1)
- net GPIO10: now also J1.5 (Pin_5), U2.10 (IO10)
- net GPIO18: now also U2.13 (IO18), USB1.A7 (Dn1), USB1.B7 (Dn2)
- net GPIO19: now also U2.14 (IO19), USB1.A6 (Dp1), USB1.B6 (Dp2)
- net GPIO2: now also U2.16 (IO2)
- net GPIO3: now also U2.15 (IO3)
- net GPIO4: now also U2.3 (IO4)
- net GPIO5: now also U2.4 (IO5)
- net GPIO6: now also J1.2 (Pin_2), U2.5 (IO6)
- net GPIO7: now also J1.1 (Pin_1), U2.6 (IO7)
- net GPIO8: now also U2.7 (IO8)
- net GPIO9: now also U2.8 (IO9)
- net UART_RXD: now also J1.4 (Pin_4), U2.11 (IO20/RXD)
- net UART_TXD: now also J1.3 (Pin_3), U2.12 (IO21/TXD)
- net at R7.1, SW3.2: now also C1.1, U2.2 (EN); no longer C1.2
- net at BZ1.1 (+): now also Q3.2 (S)
- net at R5.1: now also USB1.B5 (CC2)
- net at R6.1: now also USB1.A5 (CC1)
- net at R15.2, R16.1: now also Q3.1 (G)
- new net: R9.1, U3.6 (~{STDBY})
- new net: R8.2, U3.7 (~{CHRG})
- new net: D2.3 (K2), R9.2
- new net: D2.1 (K1), R8.1
- no-connect marks 3 -> 5
Other:
- moved on the sheet: BZ1, C1, C2, C4, C5, C7, C8, R15, R16, R7, SW3, U1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

Commit message: 基板設計中3.3v配線途中
Parts:
- added H1, H2, H3, H4: MountingHole_Pad, MountingHole:MountingHole_3.2mm_M3_ISO7380_Pad_TopBottom, symbol Mechanical:MountingHole_Pad
- SW1: value SW_Push -> SOS_Button; footprint Button_Switch_THT:SW_PUSH_6mm -> easyeda2kicad:SW-TH_4P-L12.0-W12.0-P5.00_TS-094
- SW2: value SW_Push -> Common_Button; footprint Button_Switch_THT:SW_PUSH_6mm -> easyeda2kicad:SW-TH_TS665TPZJ
- SW3: value SW_Push -> Reset_Button
Connections:
- net GND: now also H1.1, H2.1, H3.1, H4.1
- net GPIO4: now also U7.3 (SCK); no longer U7.4 (SDA)
- net GPIO5: now also U7.4 (SDA); no longer U7.3 (SCK)
